File: schematics/m5mouse/sensor.sch (KiCad schematic (older format))
At the start: 0 parts

Commit message: Add schematics
Parts:
- added C18, C19: 1u, symbol Device:C
- added D2, D3, D4, D5: SFH4550, symbol Device:LED
- added Q1, Q3, Q5, Q7: BSS138, Package_TO_SOT_SMD:SOT-23, symbol Transistor_FET:BSS138
- added Q2, Q4, Q6, Q8: ST-1KL3A, symbol Device:Q_Photo_NPN
- added R10, R12, R6, R8: 10k, symbol Device:R
- added R11, R13, R7, R9: 1k, symbol Device:R
- added R5: 33, symbol Device:R
Connections:
- new net: D3.1 (K), Q3.3 (D)
- new net: C19.1, D2.2 (A), D3.2 (A), D4.2 (A), D5.2 (A), R5.1
- new net: D4.1 (K), Q5.3 (D)
- new net: D5.1 (K), Q7.3 (D)
- new net: D2.1 (K), Q1.3 (D)
- new net +3V3: C18.1, Q2.1 (C), Q4.1 (C), Q6.1 (C), Q8.1 (C), R5.2
- new net AN_IRLED_FL: Q4.2 (E), R9.1
- new net AN_IRLED_FR: Q6.2 (E), R11.1
- new net AN_IRLED_L: Q2.2 (E), R7.1
- new net AN_IRLED_R: Q8.2 (E), R13.1
- new net GND: C18.2, C19.2, Q1.2 (S), Q3.2 (S), Q5.2 (S), Q7.2 (S), R10.2, R11.2, R12.2, R13.2, R6.2, R7.2, R8.2, R9.2
- new net IRLED_FL: Q3.1 (G), R8.1
- new net IRLED_FR: Q5.1 (G), R10.1
- new net IRLED_L: Q1.1 (G), R6.1
- new net IRLED_R: Q7.1 (G), R12.1
Other:
- note added: "1kHz pulse"
