File: schematics/m5mouse/sensor.sch (KiCad schematic (older format))
At the start: 23 parts, among them Q1 BSS138, Q2 ST-1KL3A, Q3 BSS138, Q4 ST-1KL3A, Q5 BSS138, Q6 ST-1KL3A, Q7 BSS138, Q8 ST-1KL3A

Commit message: Fix schematics
Other:
- note added: "100mA"
Changed lines of the file:
@@
 $EndComp
 Wire Wire Line
-	1200 2650 1200 2950
+	1200 2650 1200 2750
 Wire Wire Line
 	1200 3600 1200 4550
@@
 Text HLabel 10300 3850 0    50   Input ~ 0
 AN_IRLED_R
+Text Notes 2750 3600 0    50   ~ 0
+100mA
+$Comp
+L power:PWR_FLAG #FLG0105
+U 1 1 5F1AE690
+P 1650 2650
+F 0 "#FLG0105" H 1650 2725 50  0001 C CNN
+F 1 "PWR_FLAG" H 1650 2823 50  0000 C CNN
+F 2 "" H 1650 2650 50  0001 C CNN
+F 3 "~" H 1650 2650 50  0001 C CNN
+	1    1650 2650
+	1    0    0    -1
+$EndComp
+Wire Wire Line
+	1650 2650 1650 2750
+Wire Wire Line
+	1650 2750 1200 2750
+Connection ~ 1200 2750
+Wire Wire Line
+	1200 2750 1200 2950
 $EndSCHEMATC

Commit message: Put parts
Parts:
- C18, C19: value 1u -> 10u; footprint (none) -> Capacitor_SMD:C_0402_1005Metric
- D2, D3, D4, D5, Q2, Q4, Q6, Q8: footprint (none) -> Connector_PinHeader_2.54mm:PinHeader_1x02_P2.54mm_Vertical
- R10, R11, R12, R13, R5, R6, R7, R8, R9: footprint (none) -> Resistor_SMD:R_0603_1608Metric
Connections:
- net +3V3: no longer Q2.1 (C), Q4.1 (C), Q6.1 (C), Q8.1 (C)
- new net +3.3VA: Q2.1 (C), Q4.1 (C), Q6.1 (C), Q8.1 (C)
Changed lines of the file:
@@
 $Descr A4 11693 8268
 encoding utf-8
-Sheet 2 3
+Sheet 2 4
 Title ""
 Date ""
@@
 Wire Wire Line
 	3650 3600 4050 3600
-Connection ~ 1500 2950
 Wire Wire Line
 	3650 2950 3650 3200
-Wire Wire Line
-	1500 2950 3650 2950
 Wire Wire Line
 	1200 2950 1200 3300
@@
 F 0 "R7" H 4120 4346 50  0000 L CNN
 F 1 "1k" H 4120 4255 50  0000 L CNN
-F 2 "" V 3980 4300 50  0001 C CNN
+F 2 "Resistor_SMD:R_0603_1608Metric" V 3980 4300 50  0001 C CNN
 F 3 "~" H 4050 4300 50  0001 C CNN
 	1    4050 4300
@@
 F 0 "R6" H 2820 4346 50  0000 L CNN
 F 1 "10k" H 2820 4255 50  0000 L CNN
-F 2 "" V 2680 4300 50  0001 C CNN
+F 2 "Resistor_SMD:R_0603_1608Metric" V 2680 4300 50  0001 C CNN
 F 3 "~" H 2750 4300 50  0001 C CNN
 	1    2750 4300
@@
 F 0 "D2" V 3200 3800 50  0000 R CNN
 F 1 "SFH4550" V 3100 3800 50  0000 R CNN
-F 2 "" H 3150 3400 50  0001 C CNN
+F 2 "Connector_PinHeader_2.54mm:PinHeader_1x02_P2.54mm_Vertical" H 3150 3400 50  0001 C CNN
 F 3 "~" H 3150 3400 50  0001 C CNN
 	1    3150 3400
@@
 F 0 "Q2" H 3740 3446 50  0000 L CNN
 F 1 "ST-1KL3A" H 3740 3355 50  0000 L CNN
-F 2 "" H 3750 3500 50  0001 C CNN
+F 2 "Connector_PinHeader_2.54mm:PinHeader_1x02_P2.54mm_Vertical" H 3750 3500 50  0001 C CNN
 F 3 "~" H 3550 3400 50  0001 C CNN
 	1    3550 3400
 	1    0    0    -1
 $EndComp
-Wire Wire Line
-	1200 2650 1200 2750
 Wire Wire Line
 	1200 3600 1200 4550
@@
 P 2050 3450
 F 0 "C19" H 2165 3496 50  0000 L CNN
-F 1 "1u" H 2165 3405 50  0000 L CNN
-F 2 "" H 2088 3300 50  0001 C CNN
+F 1 "10u" H 2165 3405 50  0000 L CNN
+F 2 "Capacitor_SMD:C_0402_1005Metric" H 2088 3300 50  0001 C CNN
 F 3 "~" H 2050 3450 50  0001 C CNN
 	1    2050 3450
@@
 F 0 "R5" V 1750 3100 50  0000 C CNN
 F 1 "33" V 1650 3100 50  0000 C CNN
-F 2 "" V 1580 3100 50  0001 C CNN
+F 2 "Resistor_SMD:R_0603_1608Metric" V 1580 3100 50  0001 C CNN
 F 3 "~" H 1650 3100 50  0001 C CNN
 	1    1650 3100
@@
 P 1200 3450
 F 0 "C18" H 1315 3496 50  0000 L CNN
-F 1 "1u" H 1315 3405 50  0000 L CNN
-F 2 "" H 1238 3300 50  0001 C CNN
+F 1 "10u" H 1315 3405 50  0000 L CNN
+F 2 "Capacitor_SMD:C_0402_1005Metric" H 1238 3300 50  0001 C CNN
 F 3 "~" H 1200 3450 50  0001 C CNN
 	1    1200 3450
@@
 F 0 "R9" H 6270 4346 50  0000 L CNN
 F 1 "1k" H 6270 4255 50  0000 L CNN
-F 2 "" V 6130 4300 50  0001 C CNN
+F 2 "Resistor_SMD:R_0603_1608Metric" V 6130 4300 50  0001 C CNN
 F 3 "~" H 6200 4300 50  0001 C CNN
 	1    6200 4300
@@
 F 0 "R8" H 4970 4346 50  0000 L CNN
 F 1 "10k" H 4970 4255 50  0000 L CNN
-F 2 "" V 4830 4300 50  0001 C CNN
+F 2 "Resistor_SMD:R_0603_1608Metric" V 4830 4300 50  0001 C CNN
 F 3 "~" H 4900 4300 50  0001 C CNN
 	1    4900 4300
@@
 F 0 "D3" V 5350 3800 50  0000 R CNN
 F 1 "SFH4550" V 5250 3800 50  0000 R CNN
-F 2 "" H 5300 3400 50  0001 C CNN
+F 2 "Connector_PinHeader_2.54mm:PinHeader_1x02_P2.54mm_Vertical" H 5300 3400 50  0001 C CNN
 F 3 "~" H 5300 3400 50  0001 C CNN
 	1    5300 3400
@@
 F 0 "Q4" H 5890 3446 50  0000 L CNN
 F 1 "ST-1KL3A" H 5890 3355 50  0000 L CNN
-F 2 "" H 5900 3500 50  0001 C CNN
+F 2 "Connector_PinHeader_2.54mm:PinHeader_1x02_P2.54mm_Vertical" H 5900 3500 50  0001 C CNN
 F 3 "~" H 5700 3400 50  0001 C CNN
 	1    5700 3400
@@
 F 0 "R11" H 8420 4346 50  0000 L CNN
 F 1 "1k" H 8420 4255 50  0000 L CNN
-F 2 "" V 8280 4300 50  0001 C CNN
+F 2 "Resistor_SMD:R_0603_1608Metric" V 8280 4300 50  0001 C CNN
 F 3 "~" H 8350 4300 50  0001 C CNN
 	1    8350 4300
@@
 F 0 "R10" H 7120 4346 50  0000 L CNN
 F 1 "10k" H 7120 4255 50  0000 L CNN
-F 2 "" V 6980 4300 50  0001 C CNN
+F 2 "Resistor_SMD:R_0603_1608Metric" V 6980 4300 50  0001 C CNN
 F 3 "~" H 7050 4300 50  0001 C CNN
 	1    7050 4300
@@
 F 0 "D4" V 7500 3800 50  0000 R CNN
 F 1 "SFH4550" V 7400 3800 50  0000 R CNN
-F 2 "" H 7450 3400 50  0001 C CNN
+F 2 "Connector_PinHeader_2.54mm:PinHeader_1x02_P2.54mm_Vertical" H 7450 3400 50  0001 C CNN
 F 3 "~" H 7450 3400 50  0001 C CNN
 	1    7450 3400
@@
 F 0 "Q6" H 8040 3446 50  0000 L CNN
 F 1 "ST-1KL3A" H 8040 3355 50  0000 L CNN
-F 2 "" H 8050 3500 50  0001 C CNN
+F 2 "Connector_PinHeader_2.54mm:PinHeader_1x02_P2.54mm_Vertical" H 8050 3500 50  0001 C CNN
 F 3 "~" H 7850 3400 50  0001 C CNN
 	1    7850 3400
@@
 F 0 "R13" H 10570 4346 50  0000 L CNN
 F 1 "1k" H 10570 4255 50  0000 L CNN
-F 2 "" V 10430 4300 50  0001 C CNN
+F 2 "Resistor_SMD:R_0603_1608Metric" V 10430 4300 50  0001 C CNN
 F 3 "~" H 10500 4300 50  0001 C CNN
 	1    10500 4300
@@
 F 0 "R12" H 9270 4346 50  0000 L CNN
 F 1 "10k" H 9270 4255 50  0000 L CNN
-F 2 "" V 9130 4300 50  0001 C CNN
+F 2 "Resistor_SMD:R_0603_1608Metric" V 9130 4300 50  0001 C CNN
 F 3 "~" H 9200 4300 50  0001 C CNN
 	1    9200 4300
@@
 F 0 "D5" V 9650 3800 50  0000 R CNN
 F 1 "SFH4550" V 9550 3800 50  0000 R CNN
-F 2 "" H 9600 3400 50  0001 C CNN
+F 2 "Connector_PinHeader_2.54mm:PinHeader_1x02_P2.54mm_Vertical" H 9600 3400 50  0001 C CNN
 F 3 "~" H 9600 3400 50  0001 C CNN
 	1    9600 3400
@@
 F 0 "Q8" H 10190 3446 50  0000 L CNN
 F 1 "ST-1KL3A" H 10190 3355 50  0000 L CNN
-F 2 "" H 10200 3500 50  0001 C CNN
+F 2 "Connector_PinHeader_2.54mm:PinHeader_1x02_P2.54mm_Vertical" H 10200 3500 50  0001 C CNN
 F 3 "~" H 10000 3400 50  0001 C CNN
 	1    10000 3400
@@
 Wire Wire Line
 	3650 2950 5800 2950
-Connection ~ 3650 2950
 Connection ~ 5800 2950
 Wire Wire Line
@@
 100mA
 $Comp
-L power:PWR_FLAG #FLG0105
-U 1 1 5F1AE690
-P 1650 2650
-F 0 "#FLG0105" H 1650 2725 50  0001 C CNN
-F 1 "PWR_FLAG" H 1650 2823 50  0000 C CNN
-F 2 "" H 1650 2650 50  0001 C CNN
-F 3 "~" H 1650 2650 50  0001 C CNN
-	1    1650 2650
-	1    0    0    -1
-$EndComp
-Wire Wire Line
-	1650 2650 1650 2750
-Wire Wire Line
-	1650 2750 1200 2750
-Connection ~ 1200 2750
-Wire Wire Line
-	1200 2750 1200 2950
+L power:+3.3VA #PWR0112
+U 1 1 5F459E74
+P 2950 2650
+F 0 "#PWR0112" H 2950 2500 50  0001 C CNN
+F 1 "+3.3VA" H 2965 2823 50  0000 C CNN
+F 2 "" H 2950 2650 50  0001 C CNN
+F 3 "" H 2950 2650 50  0001 C CNN
+	1    2950 2650
+	1    0    0    -1
+$EndComp
+Wire Wire Line
+	2950 2650 2950 2950
+Wire Wire Line
+	2950 2950 3650 2950
+Connection ~ 3650 2950
+Wire Wire Line
+	1200 2650 1200 2950
 $EndSCHEMATC

Commit message: Adjust parts positions
Parts:
- D2, D3, D4, D5, Q2, Q4, Q6, Q8: footprint Connector_PinHeader_2.54mm:PinHeader_1x02_P2.54mm_Vertical -> m5mouse:ThroughHole_1x02_P2.54_Vertical
Changed lines of the file:
@@
 F 0 "D2" V 3200 3800 50  0000 R CNN
 F 1 "SFH4550" V 3100 3800 50  0000 R CNN
-F 2 "Connector_PinHeader_2.54mm:PinHeader_1x02_P2.54mm_Vertical" H 3150 3400 50  0001 C CNN
+F 2 "m5mouse:ThroughHole_1x02_P2.54_Vertical" H 3150 3400 50  0001 C CNN
 F 3 "~" H 3150 3400 50  0001 C CNN
 	1    3150 3400
@@
 F 0 "Q2" H 3740 3446 50  0000 L CNN
 F 1 "ST-1KL3A" H 3740 3355 50  0000 L CNN
-F 2 "Connector_PinHeader_2.54mm:PinHeader_1x02_P2.54mm_Vertical" H 3750 3500 50  0001 C CNN
+F 2 "m5mouse:ThroughHole_1x02_P2.54_Vertical" H 3750 3500 50  0001 C CNN
 F 3 "~" H 3550 3400 50  0001 C CNN
 	1    3550 3400
@@
 F 0 "D3" V 5350 3800 50  0000 R CNN
 F 1 "SFH4550" V 5250 3800 50  0000 R CNN
-F 2 "Connector_PinHeader_2.54mm:PinHeader_1x02_P2.54mm_Vertical" H 5300 3400 50  0001 C CNN
+F 2 "m5mouse:ThroughHole_1x02_P2.54_Vertical" H 5300 3400 50  0001 C CNN
 F 3 "~" H 5300 3400 50  0001 C CNN
 	1    5300 3400
@@
 F 0 "Q4" H 5890 3446 50  0000 L CNN
 F 1 "ST-1KL3A" H 5890 3355 50  0000 L CNN
-F 2 "Connector_PinHeader_2.54mm:PinHeader_1x02_P2.54mm_Vertical" H 5900 3500 50  0001 C CNN
+F 2 "m5mouse:ThroughHole_1x02_P2.54_Vertical" H 5900 3500 50  0001 C CNN
 F 3 "~" H 5700 3400 50  0001 C CNN
 	1    5700 3400
@@
 F 0 "D4" V 7500 3800 50  0000 R CNN
 F 1 "SFH4550" V 7400 3800 50  0000 R CNN
-F 2 "Connector_PinHeader_2.54mm:PinHeader_1x02_P2.54mm_Vertical" H 7450 3400 50  0001 C CNN
+F 2 "m5mouse:ThroughHole_1x02_P2.54_Vertical" H 7450 3400 50  0001 C CNN
 F 3 "~" H 7450 3400 50  0001 C CNN
 	1    7450 3400
@@
 F 0 "Q6" H 8040 3446 50  0000 L CNN
 F 1 "ST-1KL3A" H 8040 3355 50  0000 L CNN
-F 2 "Connector_PinHeader_2.54mm:PinHeader_1x02_P2.54mm_Vertical" H 8050 3500 50  0001 C CNN
+F 2 "m5mouse:ThroughHole_1x02_P2.54_Vertical" H 8050 3500 50  0001 C CNN
 F 3 "~" H 7850 3400 50  0001 C CNN
 	1    7850 3400
@@
 F 0 "D5" V 9650 3800 50  0000 R CNN
 F 1 "SFH4550" V 9550 3800 50  0000 R CNN
-F 2 "Connector_PinHeader_2.54mm:PinHeader_1x02_P2.54mm_Vertical" H 9600 3400 50  0001 C CNN
+F 2 "m5mouse:ThroughHole_1x02_P2.54_Vertical" H 9600 3400 50  0001 C CNN
 F 3 "~" H 9600 3400 50  0001 C CNN
 	1    9600 3400
@@
 F 0 "Q8" H 10190 3446 50  0000 L CNN
 F 1 "ST-1KL3A" H 10190 3355 50  0000 L CNN
-F 2 "Connector_PinHeader_2.54mm:PinHeader_1x02_P2.54mm_Vertical" H 10200 3500 50  0001 C CNN
+F 2 "m5mouse:ThroughHole_1x02_P2.54_Vertical" H 10200 3500 50  0001 C CNN
 F 3 "~" H 10000 3400 50  0001 C CNN
 	1    10000 3400

Commit message: Draw pattern
Connections:
- net GND: no longer R11.2, R13.2, R7.2, R9.2
- new net GNDA: R11.2, R13.2, R7.2, R9.2
Changed lines of the file:
@@
 Wire Wire Line
 	4050 4600 4050 4450
-$Comp
-L power:GND #PWR0119
-U 1 1 5F06F61D
-P 4050 4600
-F 0 "#PWR0119" H 4050 4350 50  0001 C CNN
-F 1 "GND" H 4055 4427 50  0000 C CNN
-F 2 "" H 4050 4600 50  0001 C CNN
-F 3 "" H 4050 4600 50  0001 C CNN
-	1    4050 4600
-	1    0    0    -1
-$EndComp
 Wire Wire Line
 	4050 3850 4050 4150
@@
 Wire Wire Line
 	6200 4600 6200 4450
-$Comp
-L power:GND #PWR0123
-U 1 1 5EF7C132
-P 6200 4600
-F 0 "#PWR0123" H 6200 4350 50  0001 C CNN
-F 1 "GND" H 6205 4427 50  0000 C CNN
-F 2 "" H 6200 4600 50  0001 C CNN
-F 3 "" H 6200 4600 50  0001 C CNN
-	1    6200 4600
-	1    0    0    -1
-$EndComp
 Wire Wire Line
 	6200 3850 6200 4150
@@
 Wire Wire Line
 	8350 4600 8350 4450
-$Comp
-L power:GND #PWR0124
-U 1 1 5EF81F14
-P 8350 4600
-F 0 "#PWR0124" H 8350 4350 50  0001 C CNN
-F 1 "GND" H 8355 4427 50  0000 C CNN
-F 2 "" H 8350 4600 50  0001 C CNN
-F 3 "" H 8350 4600 50  0001 C CNN
-	1    8350 4600
-	1    0    0    -1
-$EndComp
 Wire Wire Line
 	8350 3850 8350 4150
@@
 Wire Wire Line
 	10500 4600 10500 4450
-$Comp
-L power:GND #PWR0125
-U 1 1 5EF8828B
-P 10500 4600
-F 0 "#PWR0125" H 10500 4350 50  0001 C CNN
-F 1 "GND" H 10505 4427 50  0000 C CNN
-F 2 "" H 10500 4600 50  0001 C CNN
-F 3 "" H 10500 4600 50  0001 C CNN
-	1    10500 4600
-	1    0    0    -1
-$EndComp
 Wire Wire Line
 	10500 3850 10500 4150
@@
 Wire Wire Line
 	1200 2650 1200 2950
+$Comp
+L power:GNDA #PWR?
+U 1 1 5F495647
+P 4050 4600
+F 0 "#PWR?" H 4050 4350 50  0001 C CNN
+F 1 "GNDA" H 4055 4427 50  0000 C CNN
+F 2 "" H 4050 4600 50  0001 C CNN
+F 3 "" H 4050 4600 50  0001 C CNN
+	1    4050 4600
+	1    0    0    -1
+$EndComp
+$Comp
+L power:GNDA #PWR?
+U 1 1 5F4A60FF
+P 6200 4600
+F 0 "#PWR?" H 6200 4350 50  0001 C CNN
+F 1 "GNDA" H 6205 4427 50  0000 C CNN
+F 2 "" H 6200 4600 50  0001 C CNN
+F 3 "" H 6200 4600 50  0001 C CNN
+	1    6200 4600
+	1    0    0    -1
+$EndComp
+$Comp
+L power:GNDA #PWR?
+U 1 1 5F4A6549
+P 8350 4600
+F 0 "#PWR?" H 8350 4350 50  0001 C CNN
+F 1 "GNDA" H 8355 4427 50  0000 C CNN
+F 2 "" H 8350 4600 50  0001 C CNN
+F 3 "" H 8350 4600 50  0001 C CNN
+	1    8350 4600
+	1    0    0    -1
+$EndComp
+$Comp
+L power:GNDA #PWR?
+U 1 1 5F4A9152
+P 10500 4600
+F 0 "#PWR?" H 10500 4350 50  0001 C CNN
+F 1 "GNDA" H 10505 4427 50  0000 C CNN
+F 2 "" H 10500 4600 50  0001 C CNN
+F 3 "" H 10500 4600 50  0001 C CNN
+	1    10500 4600
+	1    0    0    -1
+$EndComp
 $EndSCHEMATC

Commit message: Fix schematics and patterns
Parts:
- C18, C19: Manf# (none) -> GRM155C80J106ME11D; URL (none) -> https://www.digikey.jp/product-detail/ja/murata-electronics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
- D2: Manf# (none) -> SFH 4550; URL (none) -> https://www.digikey.jp/product-detail/ja/osram-opto-semicon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
- Q1: Manf# (none) -> BSS138; URL (none) -> https://www.digikey.jp/product-detail/ja/on-semiconductor/B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
- Q2: Manf# (none) -> ST-1KL3A; URL (none) -> https://www.rt-shop.jp/index.php?main_page=product_info&pro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
- R10, R12, R6, R8: Manf# (none) -> RC0603FR-0710KL; URL (none) -> https://www.digikey.jp/product-detail/ja/yageo/RC0603FR-071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
- R11, R13, R7, R9: Manf# (none) -> RC0603FR-071KL; URL (none) -> https://www.digikey.jp/product-detail/ja/yageo/RC0603FR-071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
- R5: Manf# (none) -> RC0603FR-0733RL; URL (none) -> https://www.digikey.jp/product-detail/ja/yageo/RC0603FR-073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
Changed lines of the file:
@@
 F 2 "Resistor_SMD:R_0603_1608Metric" V 3980 4300 50  0001 C CNN
 F 3 "~" H 4050 4300 50  0001 C CNN
+F 4 "RC0603FR-071KL" H 4050 4300 50  0001 C CNN "Manf#"
+F 5 "https://www.digikey.jp/product-detail/ja/yageo/RC0603FR-071KL/311-1-00KHRCT-ND/729790" H 4050 4300 50  0001 C CNN "URL"
 	1    4050 4300
 	1    0    0    -1
@@
 F 2 "Resistor_SMD:R_0603_1608Metric" V 2680 4300 50  0001 C CNN
 F 3 "~" H 2750 4300 50  0001 C CNN
+F 4 "https://www.digikey.jp/product-detail/ja/yageo/RC0603FR-0710KL/311-10-0KHRCT-ND/729827" H 2750 4300 50  0001 C CNN "URL"
+F 5 "RC0603FR-0710KL" H 2750 4300 50  0001 C CNN "Manf#"
 	1    2750 4300
 	1    0    0    -1
@@
 F 2 "Package_TO_SOT_SMD:SOT-23" H 3250 4025 50  0001 L CIN
 F 3 "https://www.fairchildsemi.com/datasheets/BS/BSS138.pdf" H 3050 4100 50  0001 L CNN
+F 4 "https://www.digikey.jp/product-detail/ja/on-semiconductor/BSS138/BSS138CT-ND/244294" H 3050 4100 50  0001 C CNN "URL"
+F 5 "BSS138" H 3050 4100 50  0001 C CNN "Manf#"
 	1    3050 4100
 	1    0    0    -1
@@
 F 2 "m5mouse:ThroughHole_1x02_P2.54_Vertical" H 3150 3400 50  0001 C CNN
 F 3 "~" H 3150 3400 50  0001 C CNN
+F 4 "https://www.digikey.jp/product-detail/ja/osram-opto-semiconductors-inc/SFH-4550/475-1200-ND/806365" V 3150 3400 50  0001 C CNN "URL"
+F 5 "SFH 4550" V 3150 3400 50  0001 C CNN "Manf#"
 	1    3150 3400
 	0    -1   -1   0
@@
 F 2 "m5mouse:ThroughHole_1x02_P2.54_Vertical" H 3750 3500 50  0001 C CNN
 F 3 "~" H 3550 3400 50  0001 C CNN
+F 4 "https://www.rt-shop.jp/index.php?main_page=product_info&products_id=2746" H 3550 3400 50  0001 C CNN "URL"
+F 5 "ST-1KL3A" H 3550 3400 50  0001 C CNN "Manf#"
 	1    3550 3400
 	1    0    0    -1
@@
 F 2 "Capacitor_SMD:C_0402_1005Metric" H 2088 3300 50  0001 C CNN
 F 3 "~" H 2050 3450 50  0001 C CNN
+F 4 "GRM155C80J106ME11D" H 2050 3450 50  0001 C CNN "Manf#"
+F 5 "https://www.digikey.jp/product-detail/ja/murata-electronics/GRM155C80J106ME11D/490-13233-1-ND/5877441" H 2050 3450 50  0001 C CNN "URL"
 	1    2050 3450
 	1    0    0    -1
@@
 F 2 "Resistor_SMD:R_0603_1608Metric" V 1580 3100 50  0001 C CNN
 F 3 "~" H 1650 3100 50  0001 C CNN
+F 4 "https://www.digikey.jp/product-detail/ja/yageo/RC0603FR-0733RL/311-33-0HRCT-ND/730105" V 1650 3100 50  0001 C CNN "URL"
+F 5 "RC0603FR-0733RL" V 1650 3100 50  0001 C CNN "Manf#"
 	1    1650 3100
 	0    1    1    0
@@
 F 2 "Capacitor_SMD:C_0402_1005Metric" H 1238 3300 50  0001 C CNN
 F 3 "~" H 1200 3450 50  0001 C CNN
+F 4 "GRM155C80J106ME11D" H 1200 3450 50  0001 C CNN "Manf#"
+F 5 "https://www.digikey.jp/product-detail/ja/murata-electronics/GRM155C80J106ME11D/490-13233-1-ND/5877441" H 1200 3450 50  0001 C CNN "URL"
 	1    1200 3450
 	1    0    0    -1
@@
 F 2 "Resistor_SMD:R_0603_1608Metric" V 6130 4300 50  0001 C CNN
 F 3 "~" H 6200 4300 50  0001 C CNN
+F 4 "https://www.digikey.jp/product-detail/ja/yageo/RC0603FR-071KL/311-1-00KHRCT-ND/729790" H 6200 4300 50  0001 C CNN "URL"
+F 5 "RC0603FR-071KL" H 6200 4300 50  0001 C CNN "Manf#"
 	1    6200 4300
 	1    0    0    -1
@@
 F 2 "Resistor_SMD:R_0603_1608Metric" V 4830 4300 50  0001 C CNN
 F 3 "~" H 4900 4300 50  0001 C CNN
+F 4 "https://www.digikey.jp/product-detail/ja/yageo/RC0603FR-0710KL/311-10-0KHRCT-ND/729827" H 4900 4300 50  0001 C CNN "URL"
+F 5 "RC0603FR-0710KL" H 4900 4300 50  0001 C CNN "Manf#"
 	1    4900 4300
 	1    0    0    -1
@@
 F 2 "Resistor_SMD:R_0603_1608Metric" V 8280 4300 50  0001 C CNN
 F 3 "~" H 8350 4300 50  0001 C CNN
+F 4 "RC0603FR-071KL" H 8350 4300 50  0001 C CNN "Manf#"
+F 5 "https://www.digikey.jp/product-detail/ja/yageo/RC0603FR-071KL/311-1-00KHRCT-ND/729790" H 8350 4300 50  0001 C CNN "URL"
 	1    8350 4300
 	1    0    0    -1
@@
 F 2 "Resistor_SMD:R_0603_1608Metric" V 6980 4300 50  0001 C CNN
 F 3 "~" H 7050 4300 50  0001 C CNN
+F 4 "https://www.digikey.jp/product-detail/ja/yageo/RC0603FR-0710KL/311-10-0KHRCT-ND/729827" H 7050 4300 50  0001 C CNN "URL"
+F 5 "RC0603FR-0710KL" H 7050 4300 50  0001 C CNN "Manf#"
 	1    7050 4300
 	1    0    0    -1
@@
 F 2 "Resistor_SMD:R_0603_1608Metric" V 10430 4300 50  0001 C CNN
 F 3 "~" H 10500 4300 50  0001 C CNN
+F 4 "RC0603FR-071KL" H 10500 4300 50  0001 C CNN "Manf#"
+F 5 "https://www.digikey.jp/product-detail/ja/yageo/RC0603FR-071KL/311-1-00KHRCT-ND/729790" H 10500 4300 50  0001 C CNN "URL"
 	1    10500 4300
 	1    0    0    -1
@@
 F 2 "Resistor_SMD:R_0603_1608Metric" V 9130 4300 50  0001 C CNN
 F 3 "~" H 9200 4300 50  0001 C CNN
+F 4 "https://www.digikey.jp/product-detail/ja/yageo/RC0603FR-0710KL/311-10-0KHRCT-ND/729827" H 9200 4300 50  0001 C CNN "URL"
+F 5 "RC0603FR-0710KL" H 9200 4300 50  0001 C CNN "Manf#"
 	1    9200 4300
 	1    0    0    -1
