File: schematics/m5mouse/m5mouse.sch (KiCad schematic (older format))
At the start: 25 parts

Commit message: Add schematics
Parts:
- added C8, C9: 1p, symbol Device:C
- added D1, D6, D?: LED, symbol Device:LED
- added J3: SWD, symbol Connector_Generic:Conn_01x06
- added J6: Conn_01x03, symbol Connector_Generic:Conn_01x03
- added J7, J8: Conn_01x06, symbol Connector_Generic:Conn_01x06
- added R14: 10k, symbol Device:R
- added R15, R?: 1k, symbol Device:R
- added R4: 0, symbol Device:R
- added SW2: SW_Push, symbol Switch:SW_Push
- added Y1: 8MHz, symbol Device:Crystal_GND2
- added Y2: 32.768kHz, symbol Device:Crystal
- gave numbers to parts that had none: 25
Connections:
- net labels added: ADC2_IN0, ADC2_IN1, ADC2_IN2, ADC2_IN3, BOOT, GPIO1, GPIO2, GPIO3, GPIO4, GPIO5, GPIO6, GPIO7, GPIO8, M5_I2C1_SCL, M5_I2C1_SDA, MOT_EN, NRST, STM_I2C1_SCL, STM_I2C1_SDA, SWO, SWTCK, SWTMS, TIM1_CH1, TIM1_CH2, TIM2_CH1, TIM2_CH2, USART3_RX, USART3_TX
- net labels removed: GNDPWR, SCL, SDA
- wire segments 95 -> 202
- no-connect marks 2 -> 52
Other:
- note added: "I2C Master"
- note added: "I2C Slave"
- moved on the sheet: FB1

Commit message: schematic v0.1
Parts:
- gave numbers to parts that had none: 2
Changed lines of the file:
@@
 	8400 4700 8400 4650
-$Comp
-L power:PWR_FLAG #FLG01
-U 1 1 5F18CA87
-P 8800 4650
-F 0 "#FLG01" H 8800 4725 50  0001 C CNN
-F 1 "PWR_FLAG" H 8800 4823 50  0000 C CNN
-F 2 "" H 8800 4650 50  0001 C CNN
-F 3 "~" H 8800 4650 50  0001 C CNN
-	1    8800 4650
-	1    0    0    -1
-$EndComp
-Wire Wire Line
-	8800 4650 8800 4700
-Wire Wire Line
-	8800 4700 8400 4700
-Connection ~ 8400 4700
 $Comp
 L power:+7.5V #PWR03
@@
 Wire Wire Line
 	8400 4400 8400 4350
-$Comp
-L power:PWR_FLAG #FLG?
-U 1 1 5F2C4DE0
-P 8800 4350
-F 0 "#FLG?" H 8800 4425 50  0001 C CNN
-F 1 "PWR_FLAG" H 8800 4523 50  0000 C CNN
-F 2 "" H 8800 4350 50  0001 C CNN
-F 3 "~" H 8800 4350 50  0001 C CNN
-	1    8800 4350
-	1    0    0    -1
-$EndComp
-Wire Wire Line
-	8800 4350 8800 4400
-Wire Wire Line
-	8800 4400 8400 4400
-Connection ~ 8400 4400
 Text GLabel 11350 6700 0    50   Output ~ 0
 GPIO8
@@
 GPIO1
 $Comp
-L Device:R R?
+L Device:R R16
 U 1 1 5F34C2F2
 P 9300 7600
-F 0 "R?" H 9370 7646 50  0000 L CNN
+F 0 "R16" H 9370 7646 50  0000 L CNN
 F 1 "1k" H 9370 7555 50  0000 L CNN
 F 2 "" V 9230 7600 50  0001 C CNN
@@
 $EndComp
 $Comp
-L Device:LED D?
+L Device:LED D7
 U 1 1 5F34C2F8
 P 9300 7100
-F 0 "D?" V 9339 6982 50  0000 R CNN
+F 0 "D7" V 9339 6982 50  0000 R CNN
 F 1 "LED" V 9248 6982 50  0000 R CNN
 F 2 "" H 9300 7100 50  0001 C CNN
@@
 	9300 7250 9300 7450
 $Comp
-L power:GND #PWR?
+L power:GND #PWR09
 U 1 1 5F34C301
 P 9300 8000
-F 0 "#PWR?" H 9300 7750 50  0001 C CNN
+F 0 "#PWR09" H 9300 7750 50  0001 C CNN
 F 1 "GND" H 9305 7827 50  0000 C CNN
 F 2 "" H 9300 8000 50  0001 C CNN

Commit message: Fix schematics
Parts:
- removed D1: LED, symbol Device:LED
- added C22: 0.1, symbol Device:C
- added C23, C24: 2.2u, symbol Device:C
- added R17, R18: 10k, symbol Device:R
- L1: value INDUCTOR -> 10u
- R2: value 3.74k -> 33.2k 1%
- R3: value 10.0k -> 10.0k 1%
Connections:
- net MOT_EN is gone; now on net +5V: J8.5 (Pin_5)
- net EN: now also R17.1; no longer J7.5 (Pin_5)
- net GND: now also C22.2, C23.2, C24.2, R17.2, R18.2
- net GPIO8: now also U2.45 (PA12); no longer D6.2 (A), U2.53 (PC12)
- net NRST: now also C22.1
- net TIM2_CH2: now also U2.56 (PB4); no longer U2.28 (PB2)
- net +5V: now reaches J2.28 (Pin_28)
- net +5V: now also J7.5 (Pin_5)
- net TIM3_CH1: now reaches U2.26 (PB0)
- net TIM3_CH2: now reaches U2.27 (PB1)
- net at U2.31 (VCAP_1): now also C23.1
- net at U2.47 (VCAP_2): now also C24.1
- new net: R18.1, U2.28 (PB2)
- new net GPIO10: D6.2 (A), U2.53 (PC12)
- no-connect marks 52 -> 45
Other:
- note added: "L = (Vin - Vout) * Vout / (Vout * fsw * r * Iout)\n = (7.4 - 3.3) * 3.3 / (7.4 * 650000 * 0.3 * 1)\n = 9.376"
- note added: "Mouse Unit"
- note added: "Power Unit"
- note added: "Vout = 0.765 * (1 + R2 / R3) = 3.3\nR2 / R3 ≒ 3.32"
- note added: "boot1(Low = disable SRAM boot)"
- note added: "max1A"
- moved on the sheet: J6

Commit message: Fix schematics
Parts:
- added C26: 0.47u, symbol Device:C
- added C27: 33u, symbol Device:C
- added IC1: LM3940IMP-3.3_NOPB, SOT230P700X180-4N, symbol SamacSys_Parts:LM3940IMP-3.3_NOPB
- R2: value 33.2k 1% -> 1.07k 1%
- R3: value 10.0k 1% -> 5.9k 1%
Connections:
- net +3V3: now also J3.1 (Pin_1), C27.1, IC1.3 (OUT); no longer C5.2, C6.2, C7.2, J2.30 (Pin_30), L1.2, R2.1
- net +5V: now also C5.2, C6.2, C7.2, L1.2, R2.1, C26.1, IC1.1 (IN)
- net GND: now also C26.2, C27.2, IC1.2 (GND_1), IC1.4 (GND_2)
- net GPIO10: now also U2.52 (PC11); no longer U2.53 (PC12)
- net GPIO2: now also U2.26 (PB0); no longer U2.20 (PA4)
- net GPIO3: now also U2.27 (PB1); no longer U2.21 (PA5)
- net GPIO4: now also U2.24 (PC4); no longer U2.22 (PA6)
- net GPIO5: now also U2.25 (PC5); no longer U2.23 (PA7)
- net GPIO6: now also U2.43 (PA10); no longer U2.41 (PA8)
- net GPIO7: now also U2.44 (PA11); no longer U2.42 (PA9)
- net TIM1_CH1: now also U2.41 (PA8); no longer U2.43 (PA10)
- net TIM1_CH2: now also U2.42 (PA9); no longer U2.44 (PA11)
- net TIM3_CH1: now also U2.22 (PA6); no longer U2.26 (PB0)
- net TIM3_CH2: now also U2.23 (PA7); no longer U2.27 (PB1)
- net USART3_RX: now also U2.30 (PB11); no longer U2.58 (PB6)
- net USART3_TX: now also U2.29 (PB10); no longer U2.59 (PB7)
- net ADC2_IN0 renamed ADC1_IN0
- net ADC2_IN1 renamed ADC1_IN1
- net ADC2_IN2 renamed ADC1_IN2
- net ADC2_IN3 renamed ADC1_IN3
- net SWTCK renamed SWCLK
- net SWTMS renamed SWDIO
- net TIM2_CH1: no longer names the net of U2.50 (PA15)
- net TIM2_CH2: no longer names the net of U2.56 (PB4)
- new net TIM4_CH1: U2.58 (PB6)
- new net TIM4_CH2: U2.59 (PB7)
Other:
- note added: "L = (Vin - Vout) * Vout / (Vout * fsw * r * Iout)\n = (7.4 - 5.0) * 5.0 / (7.4 * 650000 * 0.3 * 1)\n = 8.316u"
- note added: "Vout = 0.765 * (1 + R2 / R3) = 5.0\nR2 / R3 ≒ 5.535"
- note removed: "L = (Vin - Vout) * Vout / (Vout * fsw * r * Iout)\n = (7.4 - 3.3) * 3.3 / (7.4 * 650000 * 0.3 * 1)\n = 9.376"
- note removed: "Vout = 0.765 * (1 + R2 / R3) = 3.3\nR2 / R3 ≒ 3.32"
- moved on the sheet: J6, J7, J8

Commit message: Fix schematics
Parts:
- added C28: 1u, symbol Device:C
- added D1: LED, symbol Device:LED
- added R19: 7.5k 1%, symbol Device:R
- added R20: 10k, symbol Device:R
- R17: value 10k -> 11k 1%
Connections:
- net +3V3: now also C28.1
- net +5V: now also R20.1
- net GND: now also C28.2, D1.1 (K), R19.2; no longer R17.2
- net ADC_BAT: now reaches J2.2 (Pin_2)
- net ADC_BAT: now also R17.2, R19.1
- new net: D1.2 (A), R20.2
- no-connect marks 45 -> 44
Other:
- note added: "7.4V to 3V"
- moved on the sheet: C11, C12, C14
Changed lines of the file:
@@
 L Device:C C11
 U 1 1 5EEB0B72
-P 11550 3150
-F 0 "C11" H 11665 3196 50  0000 L CNN
-F 1 "0.1u" H 11600 3050 50  0000 L CNN
-F 2 "" H 11588 3000 50  0001 C CNN
-F 3 "~" H 11550 3150 50  0001 C CNN
-	1    11550 3150
+P 11450 3150
+F 0 "C11" H 11565 3196 50  0000 L CNN
+F 1 "0.1u" H 11500 3050 50  0000 L CNN
+F 2 "" H 11488 3000 50  0001 C CNN
+F 3 "~" H 11450 3150 50  0001 C CNN
+	1    11450 3150
 	1    0    0    -1
 $EndComp
@@
 L Device:C C12
 U 1 1 5EEB2746
-P 11850 3150
-F 0 "C12" H 11965 3196 50  0000 L CNN
-F 1 "0.1u" H 11900 3050 50  0000 L CNN
-F 2 "" H 11888 3000 50  0001 C CNN
-F 3 "~" H 11850 3150 50  0001 C CNN
-	1    11850 3150
+P 11800 3150
+F 0 "C12" H 11915 3196 50  0000 L CNN
+F 1 "0.1u" H 11850 3050 50  0000 L CNN
+F 2 "" H 11838 3000 50  0001 C CNN
+F 3 "~" H 11800 3150 50  0001 C CNN
+	1    11800 3150
 	1    0    0    -1
 $EndComp
@@
 L Device:C C14
 U 1 1 5EEB2D83
-P 12450 3150
-F 0 "C14" H 12565 3196 50  0000 L CNN
-F 1 "0.1u" H 12500 3050 50  0000 L CNN
-F 2 "" H 12488 3000 50  0001 C CNN
-F 3 "~" H 12450 3150 50  0001 C CNN
-	1    12450 3150
+P 12500 3150
+F 0 "C14" H 12615 3196 50  0000 L CNN
+F 1 "0.1u" H 12550 3050 50  0000 L CNN
+F 2 "" H 12538 3000 50  0001 C CNN
+F 3 "~" H 12500 3150 50  0001 C CNN
+	1    12500 3150
 	1    0    0    -1
 $EndComp
 Wire Wire Line
-	11550 3000 11850 3000
+	11450 3000 11800 3000
 Wire Wire Line
-	11850 3000 12150 3000
-Connection ~ 11850 3000
+	11800 3000 12150 3000
+Connection ~ 11800 3000
 Wire Wire Line
-	12150 3000 12450 3000
+	12150 3000 12500 3000
 Connection ~ 12150 3000
 $Comp
@@
 $EndComp
 Wire Wire Line
-	11100 3000 11550 3000
-Connection ~ 11550 3000
+	11100 3000 11450 3000
+Connection ~ 11450 3000
 $Comp
 L Device:C C10
@@
 	11100 3000 11100 3200
 Wire Wire Line
-	11550 3300 11550 3500
+	11450 3300 11450 3500
 Wire Wire Line
-	11550 3500 12200 3500
+	11450 3500 12200 3500
 Wire Wire Line
 	12200 3500 12200 3550
 Wire Wire Line
-	11850 3300 11850 3450
+	11800 3300 11800 3450
 Wire Wire Line
-	11850 3450 12300 3450
+	11800 3450 12300 3450
 Wire Wire Line
 	12300 3450 12300 3550
@@
 	12400 3400 12400 3550
 Wire Wire Line
-	12450 3300 12500 3300
-Wire Wire Line
 	12500 3300 12500 3550
 $Comp
@@
 Wire Wire Line
 	12100 3550 12100 3600
-$Comp
-L power:+3.3V #PWR0110
-U 1 1 5EF12291
-P 10800 3450
-F 0 "#PWR0110" H 10800 3300 50  0001 C CNN
-F 1 "+3.3V" H 10815 3623 50  0000 C CNN
-F 2 "" H 10800 3450 50  0001 C CNN
-F 3 "" H 10800 3450 50  0001 C CNN
-	1    10800 3450
-	1    0    0    -1
-$EndComp
-Wire Wire Line
-	10800 3450 10800 3550
-Wire Wire Line
-	10800 3550 12100 3550
 Connection ~ 12100 3550
 $Comp
@@
 NoConn ~ 3600 3050
 NoConn ~ 3600 2950
-NoConn ~ 3600 2850
 $Comp
 L power:GND #PWR0118
@@
 Text Notes 7500 1600 0    50   ~ 0
 Mouse Unit
-Text Notes 3450 5700 0    50   ~ 0
+Text Notes 3650 5700 0    50   ~ 0
 L = (Vin - Vout) * Vout / (Vout * fsw * r * Iout)\n   = (7.4 - 5.0) * 5.0 / (7.4 * 650000 * 0.3  * 1)\n   = 8.316u
 Text Notes 5650 6000 0    50   ~ 0
@@
 P 2650 5100
 F 0 "R17" H 2720 5146 50  0000 L CNN
-F 1 "10k" H 2720 5055 50  0000 L CNN
+F 1 "11k 1%" H 2720 5055 50  0000 L CNN
 F 2 "" V 2580 5100 50  0001 C CNN
 F 3 "~" H 2650 5100 50  0001 C CNN
@@
 L power:GND #PWR010
 U 1 1 5F0AC552
-P 2650 5350
-F 0 "#PWR010" H 2650 5100 50  0001 C CNN
-F 1 "GND" H 2655 5177 50  0000 C CNN
-F 2 "" H 2650 5350 50  0001 C CNN
-F 3 "" H 2650 5350 50  0001 C CNN
-	1    2650 5350
+P 2650 5750
+F 0 "#PWR010" H 2650 5500 50  0001 C CNN
+F 1 "GND" H 2655 5577 50  0000 C CNN
+F 2 "" H 2650 5750 50  0001 C CNN
+F 3 "" H 2650 5750 50  0001 C CNN
+	1    2650 5750
 	1    0    0    -1
 $EndComp
 Wire Wire Line
-	2650 5350 2650 5250
+	2650 5350 2650 5300
 Connection ~ 2650 4850
 Wire Wire Line
@@
 Text Notes 14100 6100 0    50   ~ 0
 boot1(Low = disable SRAM boot)
-Text Notes 4800 7250 0    50   ~ 0
+Text Notes 4300 7200 0    50   ~ 0
 Vout = 0.765 * (1 + R2 / R3) = 5.0\nR2 / R3 ≒ 5.535
 $Comp
@@
 EndData
 $EndBitmap
+Text GLabel 3850 2850 2    50   Input ~ 0
+ADC_BAT
+Wire Wire Line
+	3850 2850 3600 2850
+$Comp
+L Device:R R19
+U 1 1 5F2AF41C
+P 2650 5500
+F 0 "R19" H 2720 5546 50  0000 L CNN
+F 1 "7.5k 1%" H 2720 5455 50  0000 L CNN
+F 2 "" V 2580 5500 50  0001 C CNN
+F 3 "~" H 2650 5500 50  0001 C CNN
+	1    2650 5500
+	1    0    0    -1
+$EndComp
+Wire Wire Line
+	2650 5650 2650 5750
+Text GLabel 2900 5300 2    50   Output ~ 0
+ADC_BAT
+Wire Wire Line
+	2650 5300 2900 5300
+Connection ~ 2650 5300
+Wire Wire Line
+	2650 5300 2650 5250
+Wire Wire Line
+	10800 3550 12100 3550
+$Comp
+L Device:C C28
+U 1 1 5F3E6191
+P 10450 3250
+F 0 "C28" H 10565 3296 50  0000 L CNN
+F 1 "1u" H 10565 3205 50  0000 L CNN
+F 2 "" H 10488 3100 50  0001 C CNN
+F 3 "~" H 10450 3250 50  0001 C CNN
+	1    10450 3250
+	1    0    0    -1
+$EndComp
+$Comp
+L power:GND #PWR025
+U 1 1 5F3FF633
+P 10450 3450
+F 0 "#PWR025" H 10450 3200 50  0001 C CNN
+F 1 "GND" H 10455 3277 50  0000 C CNN
+F 2 "" H 10450 3450 50  0001 C CNN
+F 3 "" H 10450 3450 50  0001 C CNN
+	1    10450 3450
+	1    0    0    -1
+$EndComp
+Wire Wire Line
+	10450 3450 10450 3400
+$Comp
+L power:+3.3V #PWR0110
+U 1 1 5EF12291
+P 10450 2900
+F 0 "#PWR0110" H 10450 2750 50  0001 C CNN
+F 1 "+3.3V" H 10465 3073 50  0000 C CNN
+F 2 "" H 10450 2900 50  0001 C CNN
+F 3 "" H 10450 2900 50  0001 C CNN
+	1    10450 2900
+	1    0    0    -1
+$EndComp
+Wire Wire Line
+	10800 3050 10800 3550
+Wire Wire Line
+	10450 2900 10450 3050
+Wire Wire Line
+	10450 3050 10800 3050
+Connection ~ 10450 3050
+Wire Wire Line
+	10450 3050 10450 3100
+$Comp
+L Device:R R20
+U 1 1 5F4F8DB4
+P 6000 6350
+F 0 "R20" H 6070 6396 50  0000 L CNN
+F 1 "10k" H 6070 6305 50  0000 L CNN
+F 2 "" V 5930 6350 50  0001 C CNN
+F 3 "~" H 6000 6350 50  0001 C CNN
+	1    6000 6350
+	1    0    0    -1
+$EndComp
+Wire Wire Line
+	6000 6050 6000 6200
+Connection ~ 6000 6050
+$Comp
+L Device:LED D1
+U 1 1 5F50B18A
+P 6000 6750
+F 0 "D1" V 6039 6632 50  0000 R CNN
+F 1 "LED" V 5948 6632 50  0000 R CNN
+F 2 "" H 6000 6750 50  0001 C CNN
+F 3 "~" H 6000 6750 50  0001 C CNN
+	1    6000 6750
+	0    -1   -1   0
+$EndComp
+Wire Wire Line
+	6000 6500 6000 6600
+$Comp
+L power:GND #PWR026
+U 1 1 5F532531
+P 6000 7050
+F 0 "#PWR026" H 6000 6800 50  0001 C CNN
+F 1 "GND" H 6005 6877 50  0000 C CNN
+F 2 "" H 6000 7050 50  0001 C CNN
+F 3 "" H 6000 7050 50  0001 C CNN
+	1    6000 7050
+	1    0    0    -1
+$EndComp
+Wire Wire Line
+	6000 7050 6000 6900
+Text Notes 3100 5200 0    50   ~ 0
+7.4V to 3V
 $EndSCHEMATC

Commit message: Put parts
Parts:
- C1, C10, C11, C12, C13, C14, C15, C16, C17, C2, C22, C23, C24, C26, C27, C28, C3, C4, C5, C6, C7, C8, C9: footprint (none) -> Capacitor_SMD:C_0402_1005Metric
- D1, D6, D7: footprint (none) -> LED_SMD:LED_0603_1608Metric
- FB1, R1, R14, R15, R16, R18, R2, R20, R3, R4: footprint (none) -> Resistor_SMD:R_0603_1608Metric
- IC1: footprint SOT230P700X180-4N -> m5mouse:LM3940IMP-3.3NOPB
- J1: footprint (none) -> Connector_JST:JST_EH_B2B-EH-A_1x02_P2.50mm_Vertical
- J2: footprint (none) -> Connector_PinHeader_2.54mm:PinHeader_2x15_P2.54mm_Vertical_SMD
- J3: footprint (none) -> Connector_JST:JST_EH_B6B-EH-A_1x06_P2.50mm_Vertical
- J6: footprint (none) -> Connector_PinHeader_2.54mm:PinHeader_1x03_P2.54mm_Vertical
- J7: footprint (none) -> Connector_PinSocket_2.54mm:PinSocket_1x06_P2.54mm_Vertical
- J8: footprint (none) -> Connector_PinHeader_2.54mm:PinHeader_1x06_P2.54mm_Vertical
- L1: footprint (none) -> Inductor_SMD:L_1008_2520Metric
- R17: value 11k 1% -> 18k 1%; footprint (none) -> Resistor_SMD:R_0603_1608Metric
- R19: value 7.5k 1% -> 10k 1%; footprint (none) -> Resistor_SMD:R_0603_1608Metric
- SW1: footprint (none) -> Button_Switch_THT:SW_E-Switch_EG1224_SPDT_Angled
- SW2: footprint (none) -> Button_Switch_THT:SW_PUSH_6mm
- Y1: footprint (none) -> m5mouse:CSTNE8M00G55Z000R0
- Y2: footprint (none) -> m5mouse:XRCGB32M768F2N10R0; symbol Device:Crystal -> Device:Crystal_GND24
Connections:
- net GND: now also Y2.2, Y2.4
- net GPIO1: now also U2.33 (PB12); no longer U2.2 (PC13)
- net GPIO10: now also U2.34 (PB13); no longer U2.52 (PC11)
- net GPIO11: now reaches U2.20 (PA4)
- net GPIO11: now also U2.52 (PC11)
- net SPI1_SCK: now reaches U2.21 (PA5)
- net at C9.1, U2.4 (PC15): now also Y2.3; no longer Y2.2
- net SPI1_CS: now reaches U2.53 (PC12)
- net SPI1_MISO: now reaches U2.56 (PB4)
- net SPI1_MOSI: now reaches U2.57 (PB5)
- no-connect marks 44 -> 38
Other:
- note added: "8.4V to 3V"
- note removed: "7.4V to 3V"
- moved on the sheet: C26, C27, C9, IC1, J1, J2, R17, R19, SW1

Commit message: Adjust parts positions
Parts:
- J1: footprint Connector_JST:JST_EH_B2B-EH-A_1x02_P2.50mm_Vertical -> Connector_JST:JST_PH_B2B-PH-K_1x02_P2.00mm_Vertical
Changed lines of the file:
@@
 F 0 "J1" H 1430 4642 50  0000 L CNN
 F 1 "Conn_01x02" H 1430 4551 50  0000 L CNN
-F 2 "Connector_JST:JST_EH_B2B-EH-A_1x02_P2.50mm_Vertical" H 1350 4650 50  0001 C CNN
+F 2 "Connector_JST:JST_PH_B2B-PH-K_1x02_P2.00mm_Vertical" H 1350 4650 50  0001 C CNN
 F 3 "~" H 1350 4650 50  0001 C CNN
 	1    1350 4650

Commit message: Draw pattern
Connections:
- net GPIO11: no longer U2.52 (PC11)
- no-connect marks 38 -> 39
Changed lines of the file:
@@
 GPIO11
 NoConn ~ 13000 5300
-Text GLabel 11350 6600 0    50   Output ~ 0
-GPIO11
-Wire Wire Line
-	11350 6600 11600 6600
 Text GLabel 11350 6700 0    50   Output ~ 0
 SPI1_CS
@@
 Wire Wire Line
 	14200 3600 15000 3600
+NoConn ~ 11600 6600
 $EndSCHEMATC
