File: schematics/m5mouse/m5mouse.kicad_pcb (KiCad board)
At the start: 2 copper layers, 110 x 50 mm, 98 parts, among them IC1 LM3940IMP-3.3_NOPB, J1 Conn_01x02, J2 M-BUS, J3 SWD, J4 Conn_02x03_Odd_Even, J5 Conn_02x03_Odd_Even, J6 Conn_01x03, J7 Conn_01x06, J8 Conn_01x06, Q1 BSS138, Q2 ST-1KL3A, Q3 BSS138, Q4 ST-1KL3A, Q5 BSS138, Q6 ST-1KL3A, Q7 BSS138, Q8 ST-1KL3A, SW1 SW_SPDT, SW2 SW_Push, U1 TPS562200, U2 STM32F405RGTx, U3 DRV8835, U4 MPU9250_9255, Y1 8MHz, Y2 32.768kHz

Commit message: Fix patterns
Parts:
- moved Ce 5.20 mm to (176.2, 112.0), turned to 225 degrees
- moved Y1 4.31 mm to (175.6, 110.0), turned to 225 degrees
- moved R4 2.04 mm to (172.4, 109.6), turned to 225 degrees
- moved FB2 2.00 mm to (179.4, 130.8)
- moved Y2 1.97 mm to (179.4, 113.4), turned to 225 degrees
- moved C8 1.28 mm to (179.0, 109.2), turned to 225 degrees
- moved R7 0.82 mm to (183.2, 127.8), turned to 270 degrees
- moved R13 0.64 mm to (147.0, 127.8), turned to 270 degrees
- renumbered C9 to Ce
Connections:
- U4 pad 25: GND -> (no net)
Routing:
- net GND: track 73.5 -> 65.5 mm, vias 79 -> 136
- net GNDA: track 81.5 -> 74.4 mm, vias 9 -> 15
- net +3.3VA: track 95.2 -> 89.3 mm
- net Net-(D5-Pad1): track 18.4 -> 13.9 mm
- net Net-(R4-Pad1): track 8.24 -> 4.30 mm
- net Net-(C8-Pad1): track 18.3 -> 15.1 mm
- net Net-(C9-Pad1): track 15.9 -> 13.2 mm
- net GPIO3: track 22.7 -> 20.3 mm
- net ADC1_IN0: track 34.1 -> 31.9 mm, vias 1 -> 2
- net Net-(U2-Pad5): track 8.21 -> 6.14 mm
- net Net-(C19-Pad1): track 66.6 -> 65.8 mm
- net SWO: track 35.4 -> 34.6 mm
- net NRST: track 36.9 -> 36.2 mm
- net ADC1_IN3: track 27.4 -> 28.1 mm
- net SWDIO: track 28.3 -> 27.7 mm
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
Commit message: Fix pattern
Parts:
- moved R4 2.41 mm to (172.2, 112.0), turned to 315 degrees
- moved Y1 1.02 mm to (175.4, 109.0)
- moved C28 0.40 mm to (174.0, 105.8)
Routing:
- net Net-(R4-Pad1): track 4.30 -> 5.38 mm
- net Net-(R4-Pad2): track 1.92 -> 2.95 mm
- net +3V3: track 189.7 -> 189.0 mm
- net Net-(C9-Pad1): track 13.2 -> 13.8 mm
- net Net-(U2-Pad5): track 6.14 -> 5.48 mm
- net GND: vias 136 -> 135

Commit message: Fix path
Parts:
- moved Y2 7.73 mm to (172.2, 110.6), turned to 270 degrees
- moved Ce 7.22 mm to (169.0, 111.4), turned to 270 degrees
- moved C10 7.00 mm to (165.4, 99.0)
- moved C11 7.00 mm to (153.9, 111.6)
- moved C12 7.00 mm to (148.6, 105.0)
- moved C13 7.00 mm to (153.8, 95.6)
- moved C14 7.00 mm to (165.4, 98.0)
- moved C15 7.00 mm to (162.3, 110.6)
- moved C16 7.00 mm to (162.3, 111.6)
- moved C17 7.00 mm to (162.3, 112.6)
- moved C18 7.00 mm to (157.1, 119.8)
- moved C19 7.00 mm to (157.1, 121.8)
- moved C20 7.00 mm to (141.0, 108.6)
- moved C21 7.00 mm to (141.0, 112.8)
- moved C22 7.00 mm to (178.8, 115.2)
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Routing:
- net SPI1_MISO: track 18.2 -> 22.9 mm
- net SWDIO: track 27.7 -> 31.6 mm
- net Net-(C8-Pad1): track 15.1 -> 12.5 mm
- net Net-(C9-Pad1): track 13.8 -> 12.5 mm
- net VIN: track 103.3 -> 102.3 mm
- net SPI1_MOSI: track 23.7 -> 22.8 mm
- net SPI1_CS: track 17.3 -> 17.8 mm
- net GND: track 65.5 -> 65.3 mm, vias 135 -> 134
Other:
- board size 110 x 50 mm -> 103 x 50 mm

Commit message: Fix pattern
Parts:
- moved C30 2.57 mm to (156.6, 118.0)
- moved C31 0.99 mm to (155.0, 116.2), turned to 270 degrees
Routing:
- net GND: track 65.3 -> 62.7 mm
- net Net-(C30-Pad1): track 4.16 -> 1.79 mm
- net +3V3: track 189.0 -> 187.5 mm
Other:
- outline, holes or cut-outs redrawn
