File: schematics/m5mouse/motor-driver.sch (KiCad schematic (older format))
At the start: 5 parts, among them J4 Conn_02x03_Odd_Even, J5 Conn_02x03_Odd_Even, U3 DRV8835

Commit message: Fix schematics
Parts:
- added C25: 10u, symbol Device:C
Connections:
- net +7.5V: now also C25.1; no longer J4.4 (Pin_4), J5.4 (Pin_4)
- net GND: now also C25.2
- net MODE: now reaches U3.11 (MODE)
- net ENBL renamed AENBL
- net AENBL: no longer U3.7 (BIN2/BENBL)
- new net +5V: J4.4 (Pin_4), J5.4 (Pin_4)
- new net BENBL: U3.7 (BIN2/BENBL)
- no-connect marks 1 -> 0
Changed lines of the file:
@@
 L power:+7.5V #PWR0127
 U 1 1 5EFE740D
-P 1950 3250
-F 0 "#PWR0127" H 1950 3100 50  0001 C CNN
-F 1 "+7.5V" H 1965 3423 50  0000 C CNN
-F 2 "" H 1950 3250 50  0001 C CNN
-F 3 "" H 1950 3250 50  0001 C CNN
-	1    1950 3250
+P 1350 3250
+F 0 "#PWR0127" H 1350 3100 50  0001 C CNN
+F 1 "+7.5V" H 1365 3423 50  0000 C CNN
+F 2 "" H 1350 3250 50  0001 C CNN
+F 3 "" H 1350 3250 50  0001 C CNN
+	1    1350 3250
 	1    0    0    -1
 $EndComp
 Wire Wire Line
-	1950 3250 2150 3250
+	1350 3250 1650 3250
 $Comp
 L power:+3.3V #PWR0128
@@
 L power:GND #PWR0130
 U 1 1 5EFEFE11
-P 2150 3600
-F 0 "#PWR0130" H 2150 3350 50  0001 C CNN
-F 1 "GND" H 2155 3427 50  0000 C CNN
-F 2 "" H 2150 3600 50  0001 C CNN
-F 3 "" H 2150 3600 50  0001 C CNN
-	1    2150 3600
+P 1900 3600
+F 0 "#PWR0130" H 1900 3350 50  0001 C CNN
+F 1 "GND" H 1905 3427 50  0000 C CNN
+F 2 "" H 1900 3600 50  0001 C CNN
+F 3 "" H 1900 3600 50  0001 C CNN
+	1    1900 3600
 	1    0    0    -1
 $EndComp
@@
 Wire Wire Line
 	2150 3250 2450 3250
-Wire Wire Line
-	4250 4100 3750 4100
-Wire Wire Line
-	4250 4100 4250 4300
-Wire Wire Line
-	4250 4300 3750 4300
-Text HLabel 4650 4100 2    50   Input ~ 0
-ENBL
-Wire Wire Line
-	4650 4100 4250 4100
-Connection ~ 4250 4100
 Text HLabel 4650 4000 2    50   Input ~ 0
 AIN
@@
 Text Label 9450 3450 0    50   ~ 0
 AOUT2
-$Comp
-L power:+7.5V #PWR0132
-U 1 1 5F14D8CD
-P 9050 3200
-F 0 "#PWR0132" H 9050 3050 50  0001 C CNN
-F 1 "+7.5V" H 9065 3373 50  0000 C CNN
-F 2 "" H 9050 3200 50  0001 C CNN
-F 3 "" H 9050 3200 50  0001 C CNN
-	1    9050 3200
-	1    0    0    -1
-$EndComp
 Wire Wire Line
 	9050 3200 9050 3450
@@
 Text Label 7500 3450 0    50   ~ 0
 BOUT2
+Wire Wire Line
+	7100 3200 7100 3450
+Text HLabel 8650 3450 0    50   Output ~ 0
+ENC_A1
+Text HLabel 8650 3950 0    50   Output ~ 0
+ENC_A2
+Wire Wire Line
+	6700 3450 7000 3450
+Wire Wire Line
+	6700 3950 7000 3950
+Text HLabel 6700 3450 0    50   Output ~ 0
+ENC_B1
+Text HLabel 6700 3950 0    50   Output ~ 0
+ENC_B2
+Wire Wire Line
+	2100 4100 2450 4100
+Wire Wire Line
+	2450 4200 2100 4200
+Wire Wire Line
+	3750 3250 4000 3250
+Text HLabel 4650 4100 2    50   Input ~ 0
+AENBL
 $Comp
-L power:+7.5V #PWR0134
-U 1 1 5F1597AC
+L power:+5V #PWR015
+U 1 1 5F24C9A0
 P 7100 3200
-F 0 "#PWR0134" H 7100 3050 50  0001 C CNN
-F 1 "+7.5V" H 7115 3373 50  0000 C CNN
+F 0 "#PWR015" H 7100 3050 50  0001 C CNN
+F 1 "+5V" H 7115 3373 50  0000 C CNN
 F 2 "" H 7100 3200 50  0001 C CNN
 F 3 "" H 7100 3200 50  0001 C CNN
@@
 	1    0    0    -1
 $EndComp
-Wire Wire Line
-	7100 3200 7100 3450
-Text HLabel 8650 3450 0    50   Output ~ 0
-ENC_A1
-Text HLabel 8650 3950 0    50   Output ~ 0
-ENC_A2
-Wire Wire Line
-	6700 3450 7000 3450
-Wire Wire Line
-	6700 3950 7000 3950
-Text HLabel 6700 3450 0    50   Output ~ 0
-ENC_B1
-Text HLabel 6700 3950 0    50   Output ~ 0
-ENC_B2
-Wire Wire Line
-	2100 4100 2450 4100
-Wire Wire Line
-	2450 4200 2100 4200
-Wire Wire Line
-	3750 3250 4000 3250
-NoConn ~ 3750 3900
+$Comp
+L power:+5V #PWR016
+U 1 1 5F24CD9E
+P 9050 3200
+F 0 "#PWR016" H 9050 3050 50  0001 C CNN
+F 1 "+5V" H 9065 3373 50  0000 C CNN
+F 2 "" H 9050 3200 50  0001 C CNN
+F 3 "" H 9050 3200 50  0001 C CNN
+	1    9050 3200
+	1    0    0    -1
+$EndComp
+Text HLabel 4650 3900 2    50   Input ~ 0
+MODE
+Wire Wire Line
+	4650 3900 3750 3900
+$Comp
+L Device:C C25
+U 1 1 5F33AAB8
+P 1650 3400
+F 0 "C25" H 1765 3446 50  0000 L CNN
+F 1 "10u" H 1765 3355 50  0000 L CNN
+F 2 "" H 1688 3250 50  0001 C CNN
+F 3 "~" H 1650 3400 50  0001 C CNN
+	1    1650 3400
+	1    0    0    -1
+$EndComp
+Connection ~ 1650 3250
+Wire Wire Line
+	1650 3250 2150 3250
+Wire Wire Line
+	1900 3600 2150 3600
+Wire Wire Line
+	1900 3600 1650 3600
+Wire Wire Line
+	1650 3600 1650 3550
+Connection ~ 1900 3600
+Wire Wire Line
+	3750 4100 4650 4100
+Text HLabel 4650 4300 2    50   Input ~ 0
+BENBL
+Wire Wire Line
+	3750 4300 4650 4300
 $EndSCHEMATC

Commit message: Put parts
Parts:
- C20, C21, C25: footprint (none) -> Capacitor_SMD:C_0402_1005Metric
- J4, J5: footprint (none) -> Connector_PinHeader_2.54mm:PinHeader_2x03_P2.54mm_Vertical
- U3: footprint (none) -> Package_SON:WSON-12-1EP_3x2mm_P0.5mm_EP1x2.65
Changed lines of the file:
@@
 $Descr A4 11693 8268
 encoding utf-8
-Sheet 3 3
+Sheet 3 4
 Title ""
 Date ""
@@
 F 0 "U3" H 3100 4519 47  0000 C CNN
 F 1 "DRV8835" H 3100 4432 47  0000 C CNN
-F 2 "" H 4700 2850 47  0001 C CNN
+F 2 "Package_SON:WSON-12-1EP_3x2mm_P0.5mm_EP1x2.65" H 4700 2850 47  0001 C CNN
 F 3 "" H 4700 2850 47  0001 C CNN
 	1    3100 4050
@@
 F 0 "C21" H 4115 3446 50  0000 L CNN
 F 1 "0.1u" H 4115 3355 50  0000 L CNN
-F 2 "" H 4038 3250 50  0001 C CNN
+F 2 "Capacitor_SMD:C_0402_1005Metric" H 4038 3250 50  0001 C CNN
 F 3 "~" H 4000 3400 50  0001 C CNN
 	1    4000 3400
@@
 F 0 "C20" H 2265 3446 50  0000 L CNN
 F 1 "0.1u" H 2265 3355 50  0000 L CNN
-F 2 "" H 2188 3250 50  0001 C CNN
+F 2 "Capacitor_SMD:C_0402_1005Metric" H 2188 3250 50  0001 C CNN
 F 3 "~" H 2150 3400 50  0001 C CNN
 	1    2150 3400
@@
 F 0 "J5" V 9146 3930 50  0000 L CNN
 F 1 "Conn_02x03_Odd_Even" V 9055 3930 50  0000 L CNN
-F 2 "" H 9050 3750 50  0001 C CNN
+F 2 "Connector_PinHeader_2.54mm:PinHeader_2x03_P2.54mm_Vertical" H 9050 3750 50  0001 C CNN
 F 3 "~" H 9050 3750 50  0001 C CNN
 	1    9050 3750
@@
 F 0 "J4" V 7196 3930 50  0000 L CNN
 F 1 "Conn_02x03_Odd_Even" V 7105 3930 50  0000 L CNN
-F 2 "" H 7100 3750 50  0001 C CNN
+F 2 "Connector_PinHeader_2.54mm:PinHeader_2x03_P2.54mm_Vertical" H 7100 3750 50  0001 C CNN
 F 3 "~" H 7100 3750 50  0001 C CNN
 	1    7100 3750
@@
 F 0 "C25" H 1765 3446 50  0000 L CNN
 F 1 "10u" H 1765 3355 50  0000 L CNN
-F 2 "" H 1688 3250 50  0001 C CNN
+F 2 "Capacitor_SMD:C_0402_1005Metric" H 1688 3250 50  0001 C CNN
 F 3 "~" H 1650 3400 50  0001 C CNN
 	1    1650 3400

Commit message: Fix schematics and patterns
Parts:
- C20: Manf# (none) -> CL05F104ZO5NNNC; URL (none) -> https://www.digikey.jp/product-detail/ja/samsung-electro-me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
- C25: Manf# (none) -> CL05A106MP8NUB8; URL (none) -> https://www.digikey.jp/product-detail/ja/samsung-electro-me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
- J4: Manf# (none) -> 929665-01-03-EU; URL (none) -> https://www.digikey.jp/product-detail/ja/3m/929665-01-03-EU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
- U3: Manf# (none) -> DRV8835DSSR; URL (none) -> https://www.digikey.jp/product-detail/ja/texas-instruments/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
Changed lines of the file:
@@
 F 2 "Package_SON:WSON-12-1EP_3x2mm_P0.5mm_EP1x2.65" H 4700 2850 47  0001 C CNN
 F 3 "" H 4700 2850 47  0001 C CNN
+F 4 "DRV8835DSSR" H 3100 4050 50  0001 C CNN "Manf#"
+F 5 "https://www.digikey.jp/product-detail/ja/texas-instruments/DRV8835DSSR/296-30391-1-ND/3188673" H 3100 4050 50  0001 C CNN "URL"
 	1    3100 4050
 	1    0    0    -1
@@
 F 2 "Capacitor_SMD:C_0402_1005Metric" H 2188 3250 50  0001 C CNN
 F 3 "~" H 2150 3400 50  0001 C CNN
+F 4 "https://www.digikey.jp/product-detail/ja/samsung-electro-mechanics/CL05F104ZO5NNNC/1276-1004-1-ND/3889090" H 2150 3400 50  0001 C CNN "URL"
+F 5 "CL05F104ZO5NNNC" H 2150 3400 50  0001 C CNN "Manf#"
 	1    2150 3400
 	1    0    0    -1
@@
 F 2 "Connector_PinHeader_2.54mm:PinHeader_2x03_P2.54mm_Vertical" H 7100 3750 50  0001 C CNN
 F 3 "~" H 7100 3750 50  0001 C CNN
+F 4 "https://www.digikey.jp/product-detail/ja/3m/929665-01-03-EU/3M156306-06-ND/3833338" V 7100 3750 50  0001 C CNN "URL"
+F 5 "929665-01-03-EU" V 7100 3750 50  0001 C CNN "Manf#"
 	1    7100 3750
 	0    1    -1   0
@@
 F 2 "Capacitor_SMD:C_0402_1005Metric" H 1688 3250 50  0001 C CNN
 F 3 "~" H 1650 3400 50  0001 C CNN
+F 4 "https://www.digikey.jp/product-detail/ja/samsung-electro-mechanics/CL05A106MP8NUB8/1276-6830-1-ND/5961689" H 1650 3400 50  0001 C CNN "URL"
+F 5 "CL05A106MP8NUB8" H 1650 3400 50  0001 C CNN "Manf#"
 	1    1650 3400
 	1    0    0    -1

Commit message: Fix pattern
Parts:
- J5: Manf# (none) -> 929665-01-03-EU; URL (none) -> https://www.digikey.jp/product-detail/ja/3m/929665-01-03-EU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
Changed lines of the file:
@@
 F 2 "Connector_PinHeader_2.54mm:PinHeader_2x03_P2.54mm_Vertical" H 9050 3750 50  0001 C CNN
 F 3 "~" H 9050 3750 50  0001 C CNN
+F 4 "929665-01-03-EU" V 9050 3750 50  0001 C CNN "Manf#"
+F 5 "https://www.digikey.jp/product-detail/ja/3m/929665-01-03-EU/3M156306-06-ND/3833338" V 9050 3750 50  0001 C CNN "URL"
 	1    9050 3750
 	0    1    -1   0
@@
 F 2 "Connector_PinHeader_2.54mm:PinHeader_2x03_P2.54mm_Vertical" H 7100 3750 50  0001 C CNN
 F 3 "~" H 7100 3750 50  0001 C CNN
-F 4 "https://www.digikey.jp/product-detail/ja/3m/929665-01-03-EU/3M156306-06-ND/3833338" V 7100 3750 50  0001 C CNN "URL"
-F 5 "929665-01-03-EU" V 7100 3750 50  0001 C CNN "Manf#"
+F 4 "929665-01-03-EU" V 7100 3750 50  0001 C CNN "Manf#"
+F 5 "https://www.digikey.jp/product-detail/ja/3m/929665-01-03-EU/3M156306-06-ND/3833338" V 7100 3750 50  0001 C CNN "URL"
 	1    7100 3750
 	0    1    -1   0
